File: embedded/schematics/schematic.sch (KiCad schematic (older format))
At the start: 53 parts

Commit message: [Feat] Completed the project schematic (Embedded)
Resolved #1.
Resolved #5.
Parts:
- removed D?: LED RED, symbol Device:LED
- removed D? (x46): LED, symbol Device:LED
- removed D?: LED GREEN, symbol Device:LED
- removed Q? (x2): BD237, Package_TO_SOT_THT:TO-126-3_Vertical, symbol Transistor_BJT:BD237
- removed R? (x2): 680, symbol Device:R
- added D? (x768): LED, symbol Device:LED
- added R? (x48): R = 221 omh, symbol Device:R
- added U? (x6): STP16CP05, symbol Driver_LED:STP16CP05
Connections:
- net labels added: +5V, Earth
- net labels removed: +12C, GND
- wire segments 75 -> 2596
Other:
- moved on the sheet: J?
